File: Documents/Kicad/Smart Ac Dimmer.kicad_sch (KiCad schematic)
At the start: 41 parts, among them J1 Conn_01x05_Socket, J2 Screw Terminal (AC Input), J3 Screw Terminal (Load), J4 Conn_01x04_Socket, Q1 BTA16-600B, U1 ESP32-C3, U2 TLP3021, U3 LF33_TO220, U4 HLK-PM01, U5 PC817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

Commit message: added the wifi ap mode. restructure the Firmware for dimmer.
Note: remove the dimmer control struct from main and complete the Web server root handler.
still remaining the R and C and restructuring the Schematic.
Parts:
- removed AE1: Antenna, symbol Device:Antenna
- removed C1, C17, C2, C3, C4, C5: C, symbol Device:C
- removed C10, C13, C14, C6: 100nF, symbol Device:C
- removed C11, C7, C9: 1uF, symbol Device:C
- removed C12: 10uF, symbol Device:C
- removed C15, C16: 15pF, symbol Device:C
- removed C8: 10nF, symbol Device:C
- removed D2: W10G, Diode_THT:Diode_Bridge_Round_D9.8mm, symbol Diode_Bridge:W10G
- removed J1: Conn_01x05_Socket, symbol Connector:Conn_01x06_Socket
- removed J2: Screw Terminal (AC Input), symbol Connector:Screw_Terminal_01x02
- removed J3: Screw Terminal (Load), symbol Connector:Screw_Terminal_01x02
- removed J4: Conn_01x04_Socket, symbol Connector:Conn_01x04_Socket
- removed Q1: BTA16-600B, Package_TO_SOT_THT:TO-220-3_Vertical, symbol Triac_Thyristor:BTA16-600B
- removed R10, R11, R12, R3, R4, R5, R6, R7, R8, R9: R, symbol Device:R
- removed R2: Potentiometer, symbol Simulation_SPICE:Potentiometer
- removed U1: ESP32-C3, Package_DFN_QFN:QFN-32-1EP_5x5mm_P0.5mm_EP3.7x3.7mm, symbol MCU_Espressif:ESP32-C3
- removed U2: TLP3021, Package_DIP:Toshiba_11-7A9, symbol Isolator:TLP3021
- removed U3: LF33_TO220, Package_TO_SOT_THT:TO-220-3_Vertical, symbol Regulator_Linear:LF33_TO220
- removed U4: HLK-PM01, Converter_ACDC:Converter_ACDC_Hi-Link_HLK-PMxx, symbol Converter_ACDC:HLK-PM01
- removed U5: PC817, Package_DIP:DIP-4_W7.62mm, symbol Isolator:PC817
- removed Y1: ABM8-40.000MHZ-B2-T, ABM8-40.000MHZ-B2-T:XTAL_ABM8-40.000MHZ-B2-T, symbol Crystal osicalltor:ABM8-40.000MHZ-B2-T
Connections:
- no-connect marks 14 -> 0
